File: Hardware/coronaampel_v2_fixed.brd (EAGLE design)
At the start: 70 x 260 mm, 155 parts, among them IC1 MH-Z19_MIRROR, IC2 TM1638, IC3 74AHCT125, IC4 LD1117AA3-A-3V3, IC5 BME680, IC6 CH340C, IC7 SCD30, IC8 OPT3001, Q1 AO3400A, Q2 AO3400A, Q3 AO3400A, Q4 AO3400A, Q5 BC848ASMD, Q6 BC848ASMD, SW1 TS1010, U1 ESP-WROOM-32, X1 XKB-U262-161N

Commit message: fixed board file, added gerbers
Parts:
- moved R24 58.4 mm to (56.2, 5.71)
- moved D2 2.84 mm to (59.1, 1.91), turned to 0 degrees
- moved C13 1.71 mm to (54.9, 2.54)
- moved R30 0.45 mm to (56.2, 7.94)
Routing:
- net EN: track 2.78 -> 7.60 mm
- net +3,3V: track 139.8 -> 143.9 mm
- net DTR: track 11.5 -> 11.0 mm
- net GND: vias 70 -> 71
Changed lines of the file:
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@@
 <element name="Q5" library="transistor-npn" package="SOT23" value="BC848ASMD" x="55.5625" y="11.1125" rot="R180"/>
 <element name="Q6" library="transistor-npn" package="SOT23" value="BC848ASMD" x="57.4675" y="16.8275"/>
-<element name="R30" library="rcl" package="R0805" value="10k" x="55.88" y="7.62" rot="R180"/>
+<element name="R30" library="rcl" package="R0805" value="10k" x="56.1975" y="7.9375" rot="R180"/>
 <element name="R31" library="rcl" package="R0805" value="10k" x="54.9275" y="14.9225" rot="R90"/>
-<element name="C13" library="rcl" package="C0805" value="22u" x="54.2925" y="4.1275" rot="R270"/>
+<element name="C13" library="rcl" package="C0805" value="22u" x="54.9275" y="2.54" rot="R270"/>
 <element name="C11" library="rcl" package="C0805" value="100n" x="68.58" y="11.43" rot="R90"/>
 <element name="BZ2" library="buzzer" package="BUZ_9_5" value="BUZZER_9mm_5mm" x="13.97" y="29.21" rot="R90"/>
 <element name="LED25" library="led" package="CHIPLED_0805" value="Blue" x="26.67" y="24.13" rot="R90"/>
 <element name="R20" library="rcl" package="R0805" value="470" x="31.115" y="24.13"/>
-<element name="D2" library="diode" package="SOD123" value="TVS 3.3V" x="56.515" y="3.175" rot="R270"/>
+<element name="D2" library="diode" package="SOD123" value="TVS 3.3V" x="59.055" y="1.905"/>
 <element name="SW1" library="switch-xkb" package="TS1010" value="TS1010" x="67.945" y="5.715" rot="R270"/>
 <element name="S1" library="switch-omron" package="B3F-10XX" value="Alert" x="65" y="249" locked="yes" rot="R270">
@@
 <element name="U$11" library="logo-htwg" package="HTWG_20" value="" x="59.055" y="153.67" rot="MR0"/>
 <element name="U$9" library="logo-htwg" package="HTWG_10" value="" x="3.175" y="89.535"/>
-<element name="R24" library="rcl" package="R0805" value="10k" x="-0.635" y="-7.62"/>
+<element name="R24" library="rcl" package="R0805" value="10k" x="56.1975" y="5.715"/>
 </elements>
 <signals>
@@
 <via x="49.53" y="7.3025" extent="1-16" drill="0.3"/>
 <via x="49.53" y="10.16" extent="1-16" drill="0.3"/>
-<via x="54.2925" y="1.5875" extent="1-16" drill="0.3"/>
+<via x="53.6575" y="1.5875" extent="1-16" drill="0.3"/>
 <via x="64.4525" y="2.8575" extent="1-16" drill="0.3"/>
 <via x="61.9125" y="9.525" extent="1-16" drill="0.3"/>
@@
 <via x="62.865" y="14.2875" extent="1-16" drill="0.3"/>
 <via x="69.215" y="5.715" extent="1-16" drill="0.3"/>
-<via x="56.515" y="3.4925" extent="1-16" drill="0.3"/>
+<via x="58.42" y="3.175" extent="1-16" drill="0.3"/>
 <via x="51.435" y="7.3025" extent="1-16" drill="0.3"/>
-<via x="58.1025" y="1.905" extent="1-16" drill="0.3"/>
+<via x="60.96" y="3.175" extent="1-16" drill="0.3"/>
 <wire x1="33.335" y1="2.8975" x2="32.385" y2="2.8975" width="0.3048" layer="1"/>
 <wire x1="32.385" y1="2.8975" x2="32.385" y2="3.81" width="0.3048" layer="1"/>
@@
 <via x="55.5625" y="30.1625" extent="1-16" drill="0.3"/>
 <via x="53.6575" y="25.7175" extent="1-16" drill="0.3"/>
+<via x="56.1975" y="0.635" extent="1-16" drill="0.3"/>
 </signal>
 <signal name="+5V">
@@
 <wire x1="61.2775" y1="4.445" x2="59.3125" y2="4.445" width="0.4064" layer="1"/>
 <wire x1="57.785" y1="27.0125" x2="57.785" y2="33.3125" width="0.6096" layer="1"/>
-<wire x1="59.3125" y1="4.445" x2="58.4175" y2="4.445" width="0.3048" layer="1"/>
 <wire x1="26.6" y1="2.94" x2="26.1175" y2="2.94" width="0.3048" layer="1"/>
 <wire x1="26.1175" y1="2.94" x2="25.4" y2="2.2225" width="0.3048" layer="1"/>
@@
 <wire x1="34.925" y1="6.985" x2="34.925" y2="6.35" width="0.3048" layer="16"/>
 <wire x1="33.335" y1="0.9525" x2="33.9725" y2="0.9525" width="0.3048" layer="1"/>
-<wire x1="53.02" y1="6.35" x2="54.2925" y2="5.0775" width="0.6096" layer="1"/>
-<wire x1="54.2925" y1="5.0775" x2="56.5125" y2="5.0775" width="0.6096" layer="1"/>
-<wire x1="56.5125" y1="5.0775" x2="56.515" y2="5.075" width="0.6096" layer="1"/>
-<wire x1="56.515" y1="5.075" x2="57.145" y2="4.445" width="0.4064" layer="1"/>
-<wire x1="57.145" y1="4.445" x2="59.3125" y2="4.445" width="0.4064" layer="1"/>
+<wire x1="58.415" y1="4.445" x2="58.4175" y2="4.445" width="0.4064" layer="1"/>
+<wire x1="58.4175" y1="4.445" x2="59.3125" y2="4.445" width="0.4064" layer="1"/>
 <wire x1="53.0225" y1="29.2075" x2="53.0225" y2="31.4325" width="0.6096" layer="1"/>
 <wire x1="53.0225" y1="31.4325" x2="54.9025" y2="33.3125" width="0.6096" layer="1"/>
 <wire x1="54.9025" y1="33.3125" x2="57.785" y2="33.3125" width="0.6096" layer="1"/>
 <contactref element="R24" pad="2"/>
-<wire x1="2.855" y1="1.2725" x2="0.315" y2="-7.62" width="0" layer="19" extent="1-1"/>
+<wire x1="53.02" y1="6.35" x2="53.6575" y2="5.7125" width="0.6096" layer="1"/>
+<wire x1="53.6575" y1="5.7125" x2="53.6575" y2="4.445" width="0.6096" layer="1"/>
+<wire x1="53.6575" y1="4.445" x2="54.6125" y2="3.49" width="0.6096" layer="1"/>
+<wire x1="54.6125" y1="3.49" x2="54.9275" y2="3.49" width="0.6096" layer="1"/>
+<wire x1="54.9275" y1="3.49" x2="57.1475" y2="3.49" width="0.6096" layer="1"/>
+<wire x1="57.1475" y1="3.49" x2="57.1475" y2="4.445" width="0.6096" layer="1"/>
+<wire x1="57.1475" y1="4.445" x2="57.1475" y2="5.715" width="0.6096" layer="1"/>
+<wire x1="57.1475" y1="3.49" x2="57.155" y2="3.49" width="0.6096" layer="1"/>
+<wire x1="57.155" y1="3.49" x2="57.155" y2="1.905" width="0.6096" layer="1"/>
+<wire x1="58.4175" y1="4.445" x2="57.1475" y2="4.445" width="0.6096" layer="1"/>
 </signal>
 <signal name="I2C_SDA">
@@
 <wire x1="58.1025" y1="15.24" x2="58.1025" y2="15.4125" width="0.3048" layer="1"/>
 <wire x1="58.1025" y1="15.4125" x2="58.4175" y2="15.7275" width="0.3048" layer="1"/>
-<wire x1="57.4675" y1="14.605" x2="57.4675" y2="8.2575" width="0.3048" layer="1"/>
-<wire x1="57.4675" y1="8.2575" x2="56.83" y2="7.62" width="0.3048" layer="1"/>
-<wire x1="59.3125" y1="8.255" x2="57.465" y2="8.255" width="0.3048" layer="1"/>
-<wire x1="57.465" y1="8.255" x2="56.83" y2="7.62" width="0.3048" layer="1"/>
+<wire x1="57.4675" y1="14.605" x2="57.4675" y2="7.9375" width="0.3048" layer="1"/>
+<wire x1="57.1475" y1="7.9375" x2="57.1475" y2="8.255" width="0.3048" layer="1"/>
+<wire x1="57.1475" y1="8.255" x2="59.3125" y2="8.255" width="0.3048" layer="1"/>
+<wire x1="57.4675" y1="7.9375" x2="57.1475" y2="7.9375" width="0.3048" layer="1"/>
 </signal>
 <signal name="N$10">
@@
 <contactref element="Q5" pad="1"/>
 <contactref element="R30" pad="2"/>
-<wire x1="56.5125" y1="12.2125" x2="56.5125" y2="9.205" width="0.3048" layer="1"/>
-<wire x1="56.5125" y1="9.205" x2="54.93" y2="7.6225" width="0.3048" layer="1"/>
-<wire x1="54.93" y1="7.6225" x2="54.93" y2="7.62" width="0.3048" layer="1"/>
+<wire x1="56.5125" y1="12.2125" x2="56.5125" y2="9.2025" width="0.3048" layer="1"/>
+<wire x1="56.5125" y1="9.2025" x2="55.2475" y2="7.9375" width="0.3048" layer="1"/>
 </signal>
 <signal name="IO0">
@@
 <contactref element="U1" pad="3"/>
 <wire x1="52.815" y1="10.08" x2="52.8825" y2="10.0125" width="0.3048" layer="1"/>
-<wire x1="52.8825" y1="10.0125" x2="55.5625" y2="10.0125" width="0.3048" layer="1"/>
+<wire x1="52.8825" y1="10.0125" x2="53.975" y2="10.0125" width="0.3048" layer="1"/>
 <contactref element="R24" pad="1"/>
-<wire x1="-1.585" y1="-7.62" x2="52.815" y2="10.08" width="0" layer="19" extent="1-1"/>
+<wire x1="53.975" y1="10.0125" x2="55.5625" y2="10.0125" width="0.3048" layer="1"/>
+<wire x1="53.975" y1="10.0125" x2="53.975" y2="6.985" width="0.3048" layer="1"/>
+<wire x1="53.975" y1="6.985" x2="53.9775" y2="6.985" width="0.3048" layer="1"/>
+<wire x1="53.9775" y1="6.985" x2="55.2475" y2="5.715" width="0.3048" layer="1"/>
 </signal>
 <signal name="N$1">
